File: ScrapHawk_FC_Main/ScrapHawk_FC_Main.kicad_sch (KiCad schematic)
At the start: 49 parts, among them IC1 MP1584EN-LF-Z, J1 USB_C_Receptacle_USB2.0_16P, J2 Conn_01x06, J3 Conn_01x06, U1 RP2040, U2 W25Q128JVS, U3 AMS1117CD-3.3, U4 LSM6DS3TR, Y1 12M

Commit message: fix capacitors size
Parts:
- removed C17: 22p, Capacitor_SMD:C_0603_1608Metric, symbol Device:C_Small
- added C1: C_Polarized, Capacitor_SMD:CP_Elec_6.3x5.2, symbol Device:C_Polarized
- C8: value 220p -> 22µF
- D2: footprint Diode_SMD:D_SMC -> Diode_SMD:D_SMB_Handsoldering
Connections:
- net +3.3V: now also C1.1
- net GND: now also C1.2
Changed lines of the file:
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@@
 	)
 	(junction
-		(at 275.59 87.63)
-		(diameter 0)
-		(color 0 0 0 0)
-	)
-	(junction
 		(at 294.64 38.1)
 		(diameter 0)
@@
 	)
 	(junction
+		(at 275.59 87.63)
+		(diameter 0)
+		(color 0 0 0 0)
+	)
+	(junction
 		(at 104.14 78.74)
 		(diameter 0)
@@
 	(wire
 		(pts
-			(xy 275.59 87.63) (xy 279.4 87.63)
+			(xy 266.7 87.63) (xy 275.59 87.63)
 		)
 		(stroke
@@
 	(wire
 		(pts
+			(xy 275.59 87.63) (xy 279.4 87.63)
+		)
+		(stroke
+			(width 0)
+			(type default)
+		)
+	)
+	(wire
+		(pts
 			(xy 114.3 78.74) (xy 124.46 78.74)
 		)
@@
 	(wire
 		(pts
-			(xy 275.59 87.63) (xy 275.59 90.17)
-		)
-		(stroke
-			(width 0)
-			(type default)
-		)
-	)
-	(wire
-		(pts
 			(xy 40.64 165.1) (xy 48.26 165.1)
 		)
@@
 	(wire
 		(pts
-			(xy 266.7 87.63) (xy 275.59 87.63)
+			(xy 124.46 69.85) (xy 124.46 71.12)
 		)
 		(stroke
@@
 	(wire
 		(pts
-			(xy 124.46 69.85) (xy 124.46 71.12)
+			(xy 43.18 19.05) (xy 48.26 19.05)
 		)
 		(stroke
@@
 	(wire
 		(pts
-			(xy 43.18 19.05) (xy 48.26 19.05)
+			(xy 270.51 49.53) (xy 285.75 49.53)
 		)
 		(stroke
@@
 	(wire
 		(pts
-			(xy 270.51 49.53) (xy 285.75 49.53)
+			(xy 270.51 57.15) (xy 270.51 58.42)
 		)
 		(stroke
@@
 	(wire
 		(pts
-			(xy 270.51 57.15) (xy 270.51 58.42)
+			(xy 175.26 81.28) (xy 175.26 80.01)
 		)
 		(stroke
@@
 	(wire
 		(pts
-			(xy 175.26 81.28) (xy 175.26 80.01)
+			(xy 275.59 96.52) (xy 275.59 97.79)
 		)
 		(stroke
@@
 	(wire
 		(pts
-			(xy 157.48 35.56) (xy 163.83 35.56)
+			(xy 275.59 87.63) (xy 275.59 88.9)
 		)
 		(stroke
@@
 	(wire
 		(pts
-			(xy 255.27 63.5) (xy 255.27 64.77)
+			(xy 157.48 35.56) (xy 163.83 35.56)
 		)
 		(stroke
@@
 	(wire
 		(pts
-			(xy 184.15 80.01) (xy 184.15 81.28)
+			(xy 255.27 63.5) (xy 255.27 64.77)
 		)
 		(stroke
@@
 	(wire
 		(pts
-			(xy 252.73 63.5) (xy 255.27 63.5)
+			(xy 184.15 80.01) (xy 184.15 81.28)
 		)
 		(stroke
@@
 	(wire
 		(pts
-			(xy 237.49 55.88) (xy 237.49 57.15)
+			(xy 252.73 63.5) (xy 255.27 63.5)
 		)
 		(stroke
@@
 	(wire
 		(pts
-			(xy 64.77 71.12) (xy 93.98 71.12)
+			(xy 237.49 55.88) (xy 237.49 57.15)
 		)
 		(stroke
@@
 	(wire
 		(pts
-			(xy 59.69 85.09) (xy 59.69 71.12)
+			(xy 64.77 71.12) (xy 93.98 71.12)
 		)
 		(stroke
@@
 	(wire
 		(pts
-			(xy 264.16 87.63) (xy 266.7 87.63)
+			(xy 59.69 85.09) (xy 59.69 71.12)
 		)
 		(stroke
@@
 	(wire
 		(pts
-			(xy 275.59 95.25) (xy 275.59 97.79)
+			(xy 264.16 87.63) (xy 266.7 87.63)
 		)
 		(stroke
@@
 			)
 		)
-		(property "Footprint" "Diode_SMD:D_SMC"
+		(property "Footprint" "Diode_SMD:D_SMB_Handsoldering"
 			(at 274.32 41.91 0)
 			(hide yes)
@@
 	(symbol
 		(lib_id "Device:C_Small")
-		(at 275.59 92.71 0)
-		(unit 1)
-		(body_style 1)
-		(exclude_from_sim no)
-		(in_bom yes)
-		(on_board yes)
-		(in_pos_files yes)
-		(dnp no)
-		(fields_autoplaced yes)
-		(property "Reference" "C17"
-			(at 278.13 91.4462 0)
-			(show_name no)
-			(do_not_autoplace no)
-			(effects
-				(font
-					(size 1.27 1.27)
-				)
-				(justify left)
-			)
-		)
-		(property "Value" "22p"
-			(at 278.13 93.9862 0)
-			(show_name no)
-			(do_not_autoplace no)
-			(effects
-				(font
-					(size 1.27 1.27)
-				)
-				(justify left)
-			)
-		)
-		(property "Footprint" "Capacitor_SMD:C_0603_1608Metric"
-			(at 275.59 92.71 0)
-			(hide yes)
-			(show_name no)
-			(do_not_autoplace no)
-			(effects
-				(font
-					(size 1.27 1.27)
-				)
-			)
-		)
-		(property "Datasheet" ""
-			(at 275.59 92.71 0)
-			(hide yes)
-			(show_name no)
-			(do_not_autoplace no)
-			(effects
-				(font
-					(size 1.27 1.27)
-				)
-			)
-		)
-		(property "Description" "Unpolarized capacitor, small symbol"
-			(at 275.59 92.71 0)
-			(hide yes)
-			(show_name no)
-			(do_not_autoplace no)
-			(effects
-				(font
-					(size 1.27 1.27)
-				)
-			)
-		)
-		(pin "1"
-		)
-		(pin "2"
-		)
-		(instances
-			(project "ScrapHawk_FC_Main"
-				(path "/000cb4d4-c35f-4b1e-baa5-bc84b3079991"
-					(reference "C17")
-					(unit 1)
-				)
-			)
-		)
-	)
-	(symbol
-		(lib_id "Device:C_Small")
 		(at 83.82 74.93 180)
 		(unit 1)
@@
 			)
 		)
-		(property "Value" "220p"
+		(property "Value" "22µF"
 			(at 229.87 39.3762 0)
 			(show_name no)
@@
 					(unit 1)
 				)
+			)
+		)
+	)
+	(symbol
+		(lib_id "Device:C_Polarized")
+		(at 275.59 92.71 0)
+		(unit 1)
+		(body_style 1)
+		(exclude_from_sim no)
+		(in_bom yes)
+		(on_board yes)
+		(in_pos_files yes)
+		(dnp no)
+		(fields_autoplaced yes)
+		(property "Reference" "C1"
+			(at 279.4 90.5509 0)
+			(show_name no)
+			(do_not_autoplace no)
+			(effects
+				(font
+					(size 1.27 1.27)
+				)
+				(justify left)
+			)
+		)
+		(property "Value" "C_Polarized"
+			(at 279.4 93.0909 0)
+			(show_name no)
+			(do_not_autoplace no)
+			(effects
+				(font
+					(size 1.27 1.27)
+				)
+				(justify left)
+			)
+		)
+		(property "Footprint" "Capacitor_SMD:CP_Elec_6.3x5.2"
+			(at 276.5552 96.52 0)
+			(hide yes)
+			(show_name no)
+			(do_not_autoplace no)
+			(effects
+				(font
+					(size 1.27 1.27)
+				)
+			)
+		)
+		(property "Datasheet" ""
+			(at 275.59 92.71 0)
+			(hide yes)
+			(show_name no)
+			(do_not_autoplace no)
+			(effects
+				(font
+					(size 1.27 1.27)
+				)
+			)
+		)
+		(property "Description" "Polarized capacitor"
+			(at 275.59 92.71 0)
+			(hide yes)
+			(show_name no)
+			(do_not_autoplace no)
+			(effects
+				(font
+					(size 1.27 1.27)
+				)
+			)
+		)
+		(pin "2"
+		)
+		(pin "1"
+		)
+		(instances
+			(project "ScrapHawk_FC_Main"
+				(path "/000cb4d4-c35f-4b1e-baa5-bc84b3079991"
+					(reference "C1")
+					(unit 1)
+				)

Commit message: update capacitor
Parts:
- added TP1, TP2: TestPoint, TestPoint:TestPoint_Pad_D1.5mm, symbol Connector:TestPoint
- C8: value 22µF -> 22uF
Connections:
- net at U1.24 (SWCLK): now also TP1.1
- net at U1.25 (SWDIO): now also TP2.1
Changed lines of the file:
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@@
+	)
+	(symbol
+		(lib_id "Connector:TestPoint")
+		(at 58.42 172.72 90)
+		(unit 1)
+		(body_style 1)
+		(exclude_from_sim no)
+		(in_bom yes)
+		(on_board yes)
+		(in_pos_files yes)
+		(dnp no)
+		(property "Reference" "TP1"
+			(at 52.07 172.72 90)
+			(show_name no)
+			(do_not_autoplace no)
+			(effects
+				(font
+					(size 1.27 1.27)
+				)
+			)
+		)
+		(property "Value" "TestPoint"
+			(at 54.61 174.752 90)
+			(hide yes)
+			(show_name no)
+			(do_not_autoplace no)
+			(effects
+				(font
+					(size 1.27 1.27)
+				)
+			)
+		)
+		(property "Footprint" "TestPoint:TestPoint_Pad_D1.5mm"
+			(at 58.42 167.64 0)
+			(hide yes)
+			(show_name no)
+			(do_not_autoplace no)
+			(effects
+				(font
+					(size 1.27 1.27)
+				)
+			)
+		)
+		(property "Datasheet" ""
+			(at 58.42 167.64 0)
+			(hide yes)
+			(show_name no)
+			(do_not_autoplace no)
+			(effects
+				(font
+					(size 1.27 1.27)
+				)
+			)
+		)
+		(property "Description" "test point"
+			(at 58.42 172.72 0)
+			(hide yes)
+			(show_name no)
+			(do_not_autoplace no)
+			(effects
+				(font
+					(size 1.27 1.27)
+				)
+			)
+		)
+		(pin "1"
+		)
+		(instances
+			(project "ScrapHawk_FC_Main"
+				(path "/000cb4d4-c35f-4b1e-baa5-bc84b3079991"
+					(reference "TP1")
+					(unit 1)
+				)
+			)
+		)
 	)
 	(symbol
@@
 	)
 	(symbol
+		(lib_id "Connector:TestPoint")
+		(at 58.42 175.26 90)
+		(unit 1)
+		(body_style 1)
+		(exclude_from_sim no)
+		(in_bom yes)
+		(on_board yes)
+		(in_pos_files yes)
+		(dnp no)
+		(property "Reference" "TP2"
+			(at 52.07 175.26 90)
+			(show_name no)
+			(do_not_autoplace no)
+			(effects
+				(font
+					(size 1.27 1.27)
+				)
+			)
+		)
+		(property "Value" "TestPoint"
+			(at 55.118 177.546 90)
+			(hide yes)
+			(show_name no)
+			(do_not_autoplace no)
+			(effects
+				(font
+					(size 1.27 1.27)
+				)
+			)
+		)
+		(property "Footprint" "TestPoint:TestPoint_Pad_D1.5mm"
+			(at 58.42 170.18 0)
+			(hide yes)
+			(show_name no)
+			(do_not_autoplace no)
+			(effects
+				(font
+					(size 1.27 1.27)
+				)
+			)
+		)
+		(property "Datasheet" ""
+			(at 58.42 170.18 0)
+			(hide yes)
+			(show_name no)
+			(do_not_autoplace no)
+			(effects
+				(font
+					(size 1.27 1.27)
+				)
+			)
+		)
+		(property "Description" "test point"
+			(at 58.42 175.26 0)
+			(hide yes)
+			(show_name no)
+			(do_not_autoplace no)
+			(effects
+				(font
+					(size 1.27 1.27)
+				)
+			)
+		)
+		(pin "1"
+		)
+		(instances
+			(project "ScrapHawk_FC_Main"
+				(path "/000cb4d4-c35f-4b1e-baa5-bc84b3079991"
+					(reference "TP2")
+					(unit 1)
+				)
+			)
+		)
+	)
+	(symbol
 		(lib_id "power:+1V1")
 		(at 121.92 85.09 270)
@@
 			)
 		)
-		(property "Value" "22µF"
+		(property "Value" "22uF"
 			(at 229.87 39.3762 0)
 			(show_name no)

Commit message: update stepdown
Parts:
- removed C15: 22p, Capacitor_SMD:C_0603_1608Metric, symbol Device:C_Small
- removed C7: 100n, Capacitor_SMD:C_0603_1608Metric, symbol Device:C_Small
- removed C8: 22uF, Capacitor_SMD:C_0603_1608Metric, symbol Device:C_Small
- removed C9: 220p, Capacitor_SMD:C_0603_1608Metric, symbol Device:C_Small
- removed D2: SS34, Diode_SMD:D_SMB_Handsoldering, symbol Device:D_Schottky
- removed IC1: MP1584EN-LF-Z, MP1584EN-LF-Z:SOIC127P600X170-9N, symbol MP1584EN:MP1584EN-LF-Z
- removed L1: 8.2uH, Inductor_SMD:L_Chilisin_BMRA00050520, symbol Device:L
- removed R5: 10K, Resistor_SMD:R_0603_1608Metric, symbol Device:R_Small
- removed R6: 52.5K, Resistor_SMD:R_0603_1608Metric, symbol Device:R_Small
- removed R7: 200K, Resistor_SMD:R_0603_1608Metric, symbol Device:R_Small
- removed R8, R9: 100K, Resistor_SMD:R_0603_1608Metric, symbol Device:R_Small
- added C17: 22u, Capacitor_SMD:C_0603_1608Metric, symbol Device:C_Small
- added C30: 0.1u, Capacitor_SMD:C_0603_1608Metric, symbol Device:C_Small
- added C31: 47u, Capacitor_SMD:C_0603_1608Metric, symbol Device:C_Small
- added L2: 4.7uH, Inductor_SMD:L_Chilisin_BMRA00050520, symbol Device:L
- added R13, R14: 52.5K, Resistor_SMD:R_0603_1608Metric, symbol Device:R_Small
- added U5: TPS562200, Package_TO_SOT_SMD:SOT-23-6, symbol Regulator_Switching:TPS562200
Connections:
- net +5V: now also C31.1, L2.2, R13.1
- net +BATT: now also C17.1, U5.3 (VIN), U5.5 (EN)
- net GND: now also C17.2, C31.2, R14.2, U5.1 (GND)
- new net: R13.2, R14.1, U5.4 (VFB)
- new net: C30.1, U5.2 (SW)
- new net: C30.2, L2.1, U5.6 (VBST)
